Commit message: Updated sawyer assets to use local pathing per recommendation https://github.com/bulletphysics/bullet3/issues/2175#issuecomment-476467882

File: assets/sawyer_description/urdf/connector_plate/connector_plate.xacro (robot description, xacro)
@@ -13,5 +13,5 @@
       <origin xyz="0 0 0" rpy="0 0 0" />
       <geometry>
-        <mesh filename="package://intera_tools_description/meshes/connector_plate/connector_plate.STL" />
+      <mesh filename="../meshes/connector_plate/connector_plate.STL" />
       </geometry>
       <material name="black">

File: assets/sawyer_description/urdf/electric_gripper/example_end_effector.urdf.xacro (robot description, xacro)
@@ -1,5 +1,5 @@
 <?xml version="1.0"?>
 <robot xmlns:xacro="http://www.ros.org/wiki/xacro" name="right_electric_gripper">
-  <xacro:include filename="$(find intera_tools_description)/urdf/electric_gripper/rethink_electric_gripper.xacro" />
+  <xacro:include filename="rethink_electric_gripper.xacro" />
   <xacro:rethink_electric_gripper side="right"
                                   l_finger="standard_narrow"

File: assets/sawyer_description/urdf/electric_gripper/fingers/basic_hard_tip.xacro (robot description, xacro)
@@ -10,5 +10,5 @@
         <origin rpy="0 0 ${pi*(g_reflect+1)/2}" xyz="0 0 0"/>
         <geometry>
-          <mesh filename="package://intera_tools_description/meshes/electric_gripper/fingers/basic_hard_tip.DAE" />
+          <mesh filename="../meshes/electric_gripper/fingers/basic_hard_tip.DAE" />
         </geometry>
       </visual>

File: assets/sawyer_description/urdf/electric_gripper/fingers/basic_soft_tip.xacro (robot description, xacro)
@@ -10,5 +10,5 @@
         <origin rpy="0 0 ${pi*(g_reflect+1)/2}" xyz="0 0 0"/>
         <geometry>
-          <mesh filename="package://intera_tools_description/meshes/electric_gripper/fingers/basic_soft_tip.DAE" />
+          <mesh filename="../meshes/electric_gripper/fingers/basic_soft_tip.DAE" />
         </geometry>
       </visual>

File: assets/sawyer_description/urdf/electric_gripper/fingers/extended_narrow.xacro (robot description, xacro)
@@ -8,5 +8,5 @@
         <origin rpy="0 0 ${-pi/2*(reflect+1)}" xyz="0 0 0"/>
         <geometry>
-          <mesh filename="package://intera_tools_description/meshes/electric_gripper/fingers/extended_narrow.DAE" />
+          <mesh filename="../meshes/electric_gripper/fingers/extended_narrow.DAE" />
         </geometry>
       </visual>
@@ -48,5 +48,5 @@
       <xacro:property name="finger_tip" value="none" scope="local"/>
     </xacro:if>
-    <xacro:include filename="$(find intera_tools_description)/urdf/electric_gripper/fingers/${finger_tip}.xacro" />
+    <xacro:include filename="electric_gripper/fingers/${finger_tip}.xacro" />
     <xacro:finger_tip_xacro parent_link="${gripper_side}_gripper_${finger_side}_finger" reflect="${reflect}" grasp="${finger_grasp}">
         <origin rpy="0 0 0" xyz="0.0 ${reflect*finger_width} ${finger_length}"/>

File: assets/sawyer_description/urdf/electric_gripper/fingers/extended_wide.xacro (robot description, xacro)
@@ -8,5 +8,5 @@
         <origin rpy="0 0 ${-pi/2*(reflect+1)}" xyz="0 0 0"/>
         <geometry>
-          <mesh filename="package://intera_tools_description/meshes/electric_gripper/fingers/extended_wide.DAE" />
+          <mesh filename="../meshes/electric_gripper/fingers/extended_wide.DAE" />
         </geometry>
       </visual>
@@ -48,5 +48,5 @@
       <xacro:property name="finger_tip" value="none" scope="local"/>
     </xacro:if>
-    <xacro:include filename="$(find intera_tools_description)/urdf/electric_gripper/fingers/${finger_tip}.xacro" />
+    <xacro:include filename="electric_gripper/fingers/${finger_tip}.xacro" />
     <xacro:finger_tip_xacro parent_link="${gripper_side}_gripper_${finger_side}_finger" reflect="${reflect}" grasp="${finger_grasp}">
         <origin rpy="0 0 0" xyz="0.0 ${reflect*finger_width} ${finger_length}"/>

File: assets/sawyer_description/urdf/electric_gripper/fingers/half_round_tip.xacro (robot description, xacro)
@@ -10,5 +10,5 @@
         <origin rpy="0 0 ${pi*(g_reflect+1)/2}" xyz="0 0 0"/>
         <geometry>
-          <mesh filename="package://intera_tools_description/meshes/electric_gripper/fingers/half_round_tip.DAE" />
+          <mesh filename="../meshes/electric_gripper/fingers/half_round_tip.DAE" />
         </geometry>
       </visual>

File: assets/sawyer_description/urdf/electric_gripper/fingers/paddle_tip.xacro (robot description, xacro)
@@ -10,5 +10,5 @@
         <origin rpy="0 0 ${pi*(g_reflect+1)/2}" xyz="0 0 0"/>
         <geometry>
-          <mesh filename="package://intera_tools_description/meshes/electric_gripper/fingers/paddle_tip.DAE" />
+	<mesh filename="../meshes/electric_gripper/fingers/paddle_tip.DAE" />
         </geometry>
       </visual>

File: assets/sawyer_description/urdf/electric_gripper/fingers/standard_narrow.xacro (robot description, xacro)
@@ -8,5 +8,5 @@
         <origin rpy="0 0 ${-pi/2*(reflect+1)}" xyz="0 0 0"/>
         <geometry>
-          <mesh filename="package://intera_tools_description/meshes/electric_gripper/fingers/standard_narrow.DAE" />
+          <mesh filename="../meshes/electric_gripper/fingers/standard_narrow.DAE" />
         </geometry>
       </visual>
@@ -19,4 +19,5 @@
           <box size="${finger_box_height} ${finger_box_width} ${finger_length}"/>
         </geometry>
+	<contact_coefficients mu="1"/>
       </collision>
       <xacro:property name="knuckle_box_height" value="0.01" scope="local"/>
@@ -48,5 +49,5 @@
       <xacro:property name="finger_tip" value="none" scope="local"/>
     </xacro:if>
-    <xacro:include filename="$(find intera_tools_description)/urdf/electric_gripper/fingers/${finger_tip}.xacro" />
+    <xacro:include filename="electric_gripper/fingers/${finger_tip}.xacro" />
     <xacro:finger_tip_xacro parent_link="${gripper_side}_gripper_${finger_side}_finger" reflect="${reflect}" grasp="${finger_grasp}">
         <origin rpy="0 0 0" xyz="0.0 ${reflect*finger_width} ${finger_length}"/>

File: assets/sawyer_description/urdf/electric_gripper/fingers/standard_wide.xacro (robot description, xacro)
@@ -8,5 +8,5 @@
         <origin rpy="0 0 ${-pi/2*(reflect+1)}" xyz="0 0 0"/>
         <geometry>
-          <mesh filename="package://intera_tools_description/meshes/electric_gripper/fingers/standard_wide.DAE" />
+          <mesh filename="../meshes/electric_gripper/fingers/standard_wide.DAE" />
         </geometry>
       </visual>
@@ -48,5 +48,5 @@
       <xacro:property name="finger_tip" value="none" scope="local"/>
     </xacro:if>
-    <xacro:include filename="$(find intera_tools_description)/urdf/electric_gripper/fingers/${finger_tip}.xacro" />
+    <xacro:include filename="electric_gripper/fingers/${finger_tip}.xacro" />
     <xacro:finger_tip_xacro parent_link="${gripper_side}_gripper_${finger_side}_finger" reflect="${reflect}" grasp="${finger_grasp}">
         <origin rpy="0 0 0" xyz="0.0 ${reflect*finger_width} ${finger_length}"/>

File: assets/sawyer_description/urdf/electric_gripper/rethink_electric_gripper.xacro (robot description, xacro)
@@ -17,5 +17,5 @@
         <origin rpy="0 0 0" xyz="0 0 0"/>
         <geometry>
-          <mesh filename="package://intera_tools_description/meshes/electric_gripper/electric_gripper_base.DAE"/>
+	<mesh filename="../meshes/electric_gripper/electric_gripper_base.DAE"/>
         </geometry>
       </visual>
@@ -47,5 +47,5 @@
      </joint>
      <!-- Connector Plate Link -->
-     <xacro:include filename="$(find intera_tools_description)/urdf/connector_plate/connector_plate.xacro" />
+     <xacro:include filename="connector_plate/connector_plate.xacro" />
      <xacro:rethink_connector_plate side="${side}" gazebo="${gazebo}"/>
      <xacro:property name="electric_gripper_parent_link" value="${side}_connector_plate_mount" scope="local"/>
@@ -60,9 +60,9 @@
     <!-- Left finger link -->
     <xacro:property name="finger_length" value="0.0" scope="global"/>
-    <xacro:include filename="$(find intera_tools_description)/urdf/electric_gripper/fingers/${l_finger}.xacro" />
+    <xacro:include filename="electric_gripper/fingers/${l_finger}.xacro" />
     <xacro:finger_xacro gripper_side="${gripper_side}" finger_side="l" reflect="1" finger_tip="${l_finger_tip}" finger_grasp="${l_finger_grasp}" gazebo="${gazebo}"/>
     <xacro:property name="tip_finger_length" value="${finger_length}" scope="local"/>
     <!-- Right finger link -->
-    <xacro:include filename="$(find intera_tools_description)/urdf/electric_gripper/fingers/${r_finger}.xacro" />
+    <xacro:include filename="electric_gripper/fingers/${r_finger}.xacro" />
     <xacro:finger_xacro gripper_side="${gripper_side}" finger_side="r" reflect="-1" finger_tip="${r_finger_tip}" finger_grasp="${r_finger_grasp}" gazebo="${gazebo}"/>
     <xacro:if value="${finger_length > tip_finger_length}">

File: assets/sawyer_description/urdf/null_gripper/example_end_effector.urdf.xacro (robot description, xacro)
@@ -1,5 +1,5 @@
 <?xml version="1.0"?>
 <robot xmlns:xacro="http://www.ros.org/wiki/xacro" name="left_null_gripper">
-  <xacro:include filename="$(find intera_tools_description)/urdf/null_gripper/null_gripper.xacro" />
+  <xacro:include filename="null_gripper/null_gripper.xacro" />
   <xacro:null_gripper side="left"/>
 </robot>

File: assets/sawyer_description/urdf/pneumatic_gripper/example_end_effector.urdf.xacro (robot description, xacro)
@@ -1,5 +1,5 @@
 <?xml version="1.0"?>
 <robot xmlns:xacro="http://www.ros.org/wiki/xacro" name="left_pneumatic_gripper">
-  <xacro:include filename="$(find intera_tools_description)/urdf/electric_gripper/rethink_pneumatic_gripper.xacro" />
+  <xacro:include filename="electric_gripper/rethink_pneumatic_gripper.xacro" />
   <xacro:rethink_pneumatic_gripper side="left"/>
 </robot>

File: assets/sawyer_description/urdf/pneumatic_gripper/pneumatic_gripper_base.xacro (robot description, xacro)
@@ -8,5 +8,5 @@
         <origin rpy="0 ${pi} ${pi}" xyz="0 0 0"/>
         <geometry>
-          <mesh filename="package://intera_tools_description/meshes/pneumatic_gripper/pneumatic_gripper_base.DAE"/>
+          <mesh filename="../meshes/pneumatic_gripper/pneumatic_gripper_base.DAE"/>
         </geometry>
       </visual>

File: assets/sawyer_description/urdf/pneumatic_gripper/rethink_pneumatic_gripper.xacro (robot description, xacro)
@@ -8,5 +8,5 @@
         <origin rpy="0 ${pi} ${pi}" xyz="0 0 0"/>
         <geometry>
-          <mesh filename="package://intera_tools_description/meshes/pneumatic_gripper/pneumatic_gripper_w_cup.DAE"/>
+          <mesh filename="../meshes/pneumatic_gripper/pneumatic_gripper_w_cup.DAE"/>
         </geometry>
       </visual>

File: assets/sawyer_description/urdf/sawyer.urdf.xacro (robot description, xacro)
@@ -4,12 +4,12 @@
   <xacro:arg name="pedestal" default="true"/>
   <xacro:arg name="static" default="true"/>
-  <xacro:arg name="electric_gripper" default="false"/>
+  <xacro:arg name="electric_gripper" default="true"/>
   <!-- Sawyer Base URDF -->
-  <xacro:include filename="$(find sawyer_description)/urdf/sawyer_base.urdf.xacro">
+  <xacro:include filename="sawyer_base.urdf.xacro">
     <xacro:arg name="gazebo" value="${gazebo}"/>
     <xacro:arg name="pedestal" value="${pedestal}"/>
   </xacro:include>
   <xacro:if value="$(arg gazebo)">
-  <xacro:include filename="$(find sawyer_description)/urdf/sawyer_base.gazebo.xacro">
+  <xacro:include filename="sawyer_base.gazebo.xacro">
     <xacro:arg name="static" value="${static}"/>
     <xacro:arg name="pedestal" value="${pedestal}"/>
@@ -18,5 +18,5 @@
   <!-- Electric Gripper End Effector -->
   <xacro:if value="$(arg electric_gripper)">
-  <xacro:include filename="$(find sawyer_description)/urdf/sawyer_electric_gripper.urdf.xacro">
+  <xacro:include filename="sawyer_electric_gripper.urdf.xacro">
     <xacro:arg name="gazebo" value="${gazebo}"/>
   </xacro:include>

File: assets/sawyer_description/urdf/sawyer_electric_gripper.urdf.xacro (robot description, xacro)
@@ -8,5 +8,5 @@
     <xacro:property name="gazebo_tag" value="false" scope="local"/>
   </xacro:unless>
-  <xacro:include filename="$(find intera_tools_description)/urdf/electric_gripper/rethink_electric_gripper.xacro" />
+  <xacro:include filename="electric_gripper/rethink_electric_gripper.xacro" />
   <xacro:rethink_electric_gripper side="right"
                                   gazebo="${gazebo_tag}"

File: assets/sawyer_description/urdf/sawyer_static.urdf (robot description, URDF)
Before this commit: robot sawyer, 36 links, 35 joints
Links:
- removed link head_camera_optical
- removed link right_hand_camera_optical
- removed link world
- link head: geometry collision sphere radius=0.18; visual mesh filename=package://sawyer_description/meshes/sawyer_pv/head.DAE
- link pedestal: geometry collision cylinder length=0.62 radius=0.18; visual mesh filename=package://sawyer_description/meshes/sawyer_pv/pedestal.DAE
- link right_arm_base_link: geometry collision cylinder length=0.24 radius=0.08; visual mesh filename=package://sawyer_description/meshes/sawyer_pv/base.DAE
- link right_arm_itb: mass None -> 0.0001
- link right_connector_plate_base: geometry collision cylinder length=0.0302 radius=0.04; visual mesh filename=../meshes/connector_plate/connector_plate.STL
- link right_electric_gripper_base: geometry collision cylinder length=0.1 radius=0.029; visual mesh filename=../meshes/electric_gripper/electric_gripper_base.DAE
- link right_gripper_l_finger: geometry collision box size=0.01 0.0135 0.075; collision box size=0.01 0.05 0.017
- link right_gripper_l_finger_tip: geometry collision box size=0.016 0.007 0.037; visual mesh filename=../meshes/electric_gripper/fingers/basic_soft_tip.DAE
- link right_gripper_r_finger: geometry collision box size=0.01 0.0135 0.075; collision box size=0.01 0.05 0.017
- link right_gripper_r_finger_tip: geometry collision box size=0.016 0.007 0.037; visual mesh filename=../meshes/electric_gripper/fingers/basic_soft_tip.DAE
- link right_hand: mass 0.01 -> 1.0E-08
- link right_l0: geometry collision sphere radius=0.07; visual mesh filename=package://sawyer_description/meshes/sawyer_mp3/l0.DAE
- link right_l1: geometry collision sphere radius=0.07; visual mesh filename=package://sawyer_description/meshes/sawyer_mp3/l1.DAE
- link right_l1_2: mass None -> 1.0E-08
- link right_l2: geometry collision cylinder length=0.34 radius=0.06; visual mesh filename=package://sawyer_description/meshes/sawyer_pv/l2.DAE
- link right_l2_2: mass None -> 1.0E-08
- link right_l3: geometry collision sphere radius=0.06; visual mesh filename=package://sawyer_description/meshes/sawyer_pv/l3.DAE
- link right_l4: geometry collision cylinder length=0.30 radius=0.045; visual mesh filename=package://sawyer_description/meshes/sawyer_pv/l4.DAE
- link right_l4_2: mass None -> 1.0E-08
- link right_l5: geometry collision sphere radius=0.06; visual mesh filename=package://sawyer_description/meshes/sawyer_pv/l5.DAE
- link right_l6: geometry collision cylinder length=0.05 radius=0.055; visual mesh filename=package://sawyer_description/meshes/sawyer_mp1/l6.DAE
- link right_torso_itb: mass None -> 0.0001
- link screen: mass None -> 0.0001
- link torso: mass None -> 0.0001
Joints:
- removed joint fixed
- removed joint head_camera_optical_joint
- removed joint right_hand_camera_optical_joint
- joint right_j6: limit lower=-3.14 upper=3.14 effort=9.0 velocity=4.545 -> lower=-4.7124 upper=4.7124 effort=9.0 velocity=4.545
