Commit message: Fixed IK to work independently of URDF loading policy (e.g., with/without merged links). Made Sawyer base 1160kg instead of 60kg to prevent tipping.

File: assets/sawyer_description/urdf/sawyer_base.urdf.xacro (robot description, xacro)
@@ -54,5 +54,5 @@
     <inertial>
       <origin rpy="0 0 0" xyz="0 0 -0.5"/>
-      <mass value="60.86397744"/>
+      <mass value="1160.86397744"/>
       <inertia ixx="5.0635929" ixy="0.00103417" ixz="0.80199628" iyy="6.08689388" iyz="0.00105311" izz="4.96191932"/>
     </inertial>

File: assets/sawyer_description/urdf/sawyer_static.urdf (robot description, URDF)
Before this commit: robot sawyer, 33 links, 32 joints
Links:
- link pedestal: mass 60.86397744 -> 1160.86397744
