Commit message: Added set_timestep to Simulator. Added Sensor base class and LaserRangeFinder example. Sensors attached to robots hasn't been tested yet.

File: assets/sawyer_description/urdf/electric_gripper/fingers/basic_hard_tip.xacro (robot description, xacro)
@@ -10,5 +10,5 @@
         <origin rpy="0 0 ${pi*(g_reflect+1)/2}" xyz="0 0 0"/>
         <geometry>
-          <mesh filename="../meshes/electric_gripper/fingers/basic_hard_tip.DAE" />
+          <mesh filename="package://sawyer_description/meshes/electric_gripper/fingers/basic_hard_tip.DAE" />
         </geometry>
       </visual>

File: assets/sawyer_description/urdf/electric_gripper/fingers/basic_soft_tip.xacro (robot description, xacro)
@@ -10,5 +10,5 @@
         <origin rpy="0 0 ${pi*(g_reflect+1)/2}" xyz="0 0 0"/>
         <geometry>
-          <mesh filename="../meshes/electric_gripper/fingers/basic_soft_tip.DAE" />
+          <mesh filename="package://sawyer_description/meshes/electric_gripper/fingers/basic_soft_tip.DAE" />
         </geometry>
       </visual>

File: assets/sawyer_description/urdf/electric_gripper/fingers/standard_narrow.xacro (robot description, xacro)
@@ -8,5 +8,5 @@
         <origin rpy="0 0 ${-pi/2*(reflect+1)}" xyz="0 0 0"/>
         <geometry>
-          <mesh filename="../meshes/electric_gripper/fingers/standard_narrow.DAE" />
+          <mesh filename="package://sawyer_description/meshes/electric_gripper/fingers/standard_narrow.DAE" />
         </geometry>
       </visual>

File: assets/sawyer_description/urdf/electric_gripper/rethink_electric_gripper.xacro (robot description, xacro)
@@ -17,5 +17,5 @@
         <origin rpy="0 0 0" xyz="0 0 0"/>
         <geometry>
-	<mesh filename="../meshes/electric_gripper/electric_gripper_base.DAE"/>
+	<mesh filename="package://sawyer_description/meshes/electric_gripper/electric_gripper_base.DAE"/>
         </geometry>
       </visual>

File: assets/sawyer_description/urdf/sawyer.urdf.xacro (robot description, xacro)
@@ -10,15 +10,7 @@
     <xacro:arg name="pedestal" value="${pedestal}"/>
   </xacro:include>
-  <xacro:if value="$(arg gazebo)">
-  <xacro:include filename="sawyer_base.gazebo.xacro">
-    <xacro:arg name="static" value="${static}"/>
-    <xacro:arg name="pedestal" value="${pedestal}"/>
-  </xacro:include>
-  </xacro:if>
   <!-- Electric Gripper End Effector -->
-  <xacro:if value="$(arg electric_gripper)">
   <xacro:include filename="sawyer_electric_gripper.urdf.xacro">
     <xacro:arg name="gazebo" value="${gazebo}"/>
   </xacro:include>
-  </xacro:if>
 </robot>

File: assets/sawyer_description/urdf/sawyer_base.urdf.xacro (robot description, xacro)
@@ -18,5 +18,11 @@
     <color rgba="0.75294 0.75294 0.75294 1"/>
   </material>
-  <link name="base"/>
+  <link name="base">
+    <inertial>
+      <origin rpy="0 0 0" xyz="-0.1 0 0.07"/>
+      <mass value=".0"/>
+      <inertia ixx="0.05" ixy="0" ixz="0" iyy="0.06" iyz="0" izz="0.03"/>
+    </inertial>
+  </link>
   <link name="torso">
     <visual>

File: assets/sawyer_description/urdf/sawyer_static.urdf (robot description, URDF)
Before this commit: robot sawyer, 33 links, 32 joints
Links:
- removed link controller_box
- removed link pedestal_feet
- removed link right_l1_2
- removed link right_l2_2
- removed link right_l4_2
- link base: mass None -> .0
- link head: geometry collision sphere radius=0.18; visual mesh filename=package://sawyer_description/meshes/sawyer_pv/head.STL
- link pedestal: mass 1160.86397744 -> 60.864
- link right_connector_plate_base: geometry collision cylinder length=0.0302 radius=0.04; visual mesh filename=package://sawyer_description/meshes/connector_plate/connect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
- link right_electric_gripper_base: geometry collision cylinder length=0.1 radius=0.029; visual mesh filename=package://sawyer_description/meshes/electric_gripper/electr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
- link right_gripper_l_finger: geometry collision box size=0.01 0.0135 0.075; collision box size=0.01 0.05 0.017
- link right_gripper_l_finger_tip: geometry collision box size=0.016 0.007 0.037; visual mesh filename=package://sawyer_description/meshes/electric_gripper/finger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
- link right_gripper_r_finger: geometry collision box size=0.01 0.0135 0.075; collision box size=0.01 0.05 0.017
- link right_gripper_r_finger_tip: geometry collision box size=0.016 0.007 0.037; visual mesh filename=package://sawyer_description/meshes/electric_gripper/finger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
- link right_hand: mass 1.0E-08 -> 1e-08; geometry collision cylinder length=0 radius=0
- link right_l2: mass 1.745 -> 1.7251; geometry collision cylinder length=0.35 radius=0.06; visual mesh filename=package://sawyer_description/meshes/sawyer_pv/l2.DAE
- link right_l3: mass 2.5097 -> 2.4743
- link right_l4: mass 1.1136 -> 1.0433; geometry collision cylinder length=0.36 radius=0.045; visual mesh filename=package://sawyer_description/meshes/sawyer_pv/l4.DAE
- link right_l5: mass 1.5625 -> 1.5343; geometry collision sphere radius=0.06; visual mesh filename=package://sawyer_description/meshes/sawyer_pv/l5.STL
- link right_l6: geometry collision cylinder length=0.05 radius=0.065; visual mesh filename=package://sawyer_description/meshes/sawyer_mp1/l6.STL
- link torso: geometry visual box size=0 0 0
Joints:
- removed joint controller_box_fixed
- removed joint pedestal_feet_fixed
- removed joint right_j1_2
- removed joint right_j2_2
- removed joint right_j4_2
- joint display_joint: origin xyz=0.03 0.0 0.105 rpy=1.57079632679 0 1.57079632679 -> xyz=0.03 0 0.105 rpy=1.5708 0 1.5708
- joint head_camera: origin xyz=0.0228027 0 0.216572 rpy=-2.1293 0 -1.57079632679 -> xyz=0.022803 0 0.21657 rpy=-2.1293 0 -1.5708
- joint head_pan: limit lower=-5.0952 upper=0.9064 effort=8 velocity=1.8 -> lower=-5.1477 upper=0.9559 effort=8 velocity=1.8
- joint pedestal_fixed: origin xyz=0.0 0.0 0.0 rpy=0 0 0 -> xyz=0 0 0 rpy=0 0 0
- joint right_arm_itb: origin xyz=-.055 0 .075 rpy=0 -1.57079632679 0 -> xyz=-0.055 0 0.075 rpy=0 -1.5708 0
- joint right_arm_mount: origin xyz=0.0 0.0 0.0 rpy=0 0 0 -> xyz=0 0 0 rpy=0 0 0
- joint right_hand: origin xyz=0 0 0.0245 rpy=0 0 1.570796 -> xyz=0 0 0.0245 rpy=0 0 1.5708
- joint right_hand_camera: origin xyz=0.039552 -0.033 0.0695 rpy=0 1.57079632679 0 -> xyz=0.039552 -0.033 0.0695 rpy=0 1.5708 0
- joint right_j0: limit lower=-3.0503 upper=3.0503 effort=80.0 velocity=1.74 -> lower=-3.0503 upper=3.0503 effort=80 velocity=1.74
- joint right_j1: limit lower=-3.8095 upper=2.2736 effort=80.0 velocity=1.328 -> lower=-3.8183 upper=2.2824 effort=80 velocity=1.328; origin xyz=0.081 0.05 0.237 rpy=-1.57079632679 1.57079632679 0 -> xyz=0.081 0.05 0.237 rpy=-1.5708 1.5708 0
- joint right_j2: limit lower=-3.0426 upper=3.0426 effort=40.0 velocity=1.957 -> lower=-3.0514 upper=3.0514 effort=40 velocity=1.957; origin xyz=0 -0.14 0.1425 rpy=1.57079632679 0 0 -> xyz=0 -0.14 0.1425 rpy=1.5708 0 0
- joint right_j3: limit lower=-3.0439 upper=3.0439 effort=40.0 velocity=1.957 -> lower=-3.0514 upper=3.0514 effort=40 velocity=1.957; origin xyz=0 -0.042 0.26 rpy=-1.57079632679 0 0 -> xyz=0 -0.042 0.26 rpy=-1.5708 0 0
- joint right_j4: limit lower=-2.9761 upper=2.9761 effort=9.0 velocity=3.485 -> lower=-2.9842 upper=2.9842 effort=9 velocity=3.485; origin xyz=0 -0.125 -0.1265 rpy=1.57079632679 0 0 -> xyz=0 -0.125 -0.1265 rpy=1.5708 0 0
- joint right_j5: limit lower=-2.9761 upper=2.9761 effort=9.0 velocity=3.485 -> lower=-2.9842 upper=2.9842 effort=9 velocity=3.485; origin xyz=0 0.031 0.275 rpy=-1.57079632679 0 0 -> xyz=0 0.031 0.275 rpy=-1.5708 0 0
- joint right_j6: limit lower=-4.7124 upper=4.7124 effort=9.0 velocity=4.545 -> lower=-4.7104 upper=4.7104 effort=9 velocity=4.545; origin xyz=0 -0.11 0.1053 rpy=-1.57079632679 -0.17453 3.1416 -> xyz=0 -0.11 0.1053 rpy=-1.5708 -0.17453 3.1416
- joint right_torso_itb: origin xyz=-.055 0 .22 rpy=0 -1.57079632679 0 -> xyz=-0.055 0 0.22 rpy=0 -1.5708 0
- joint right_wrist: origin xyz=0 0 0.10541 rpy=1.57079632679 0 0 -> xyz=0 0 0.10541 rpy=1.5708 0 0
